Commit message: Update allegro_hand_digit_right.urdf

File: allegro_hand_digit_right.urdf (robot description, URDF)
Before this commit: robot allegro_hand_right, 21 links, 20 joints
Links:
- link base_link: geometry collision mesh filename=allegro_digit/collision/base_link_merged.STL; visual mesh filename=allegro_digit/stl/base_link.STL
- link link_0.0: geometry collision mesh filename=allegro_digit/collision/link_0.0_merged.STL; visual mesh filename=allegro_digit/stl/link_0.0.STL
- link link_1.0: geometry collision mesh filename=allegro_digit/collision/link_1.0_merged.STL; visual mesh filename=allegro_digit/stl/link_1.0.STL
- link link_10.0: geometry collision mesh filename=allegro_digit/collision/link_2.0_merged.STL; visual mesh filename=allegro_digit/stl/link_2.0.STL
- link link_11.0: geometry collision mesh filename=allegro_digit/collision/link_3.0_merged.STL; visual mesh filename=allegro_digit/stl/link_3.0.STL
- link link_11.0_tip: geometry collision mesh filename=allegro_digit/collision/digit.STL; visual mesh filename=allegro_digit/stl/digit.STL
- link link_12.0: geometry collision mesh filename=allegro_digit/collision/link_12.0_right_merged.STL; visual mesh filename=allegro_digit/stl/link_12.0_right.STL
- link link_13.0: geometry collision mesh filename=allegro_digit/collision/link_13.0_merged.STL; visual mesh filename=allegro_digit/stl/link_13.0.STL
- link link_14.0: geometry collision mesh filename=allegro_digit/stl/link_14.0_merged.STL; visual mesh filename=allegro_digit/stl/link_14.0.STL
- link link_15.0: geometry collision mesh filename=allegro_digit/stl/link_15.0_merged.STL; visual mesh filename=allegro_digit/stl/link_15.0.STL
- link link_15.0_tip: geometry collision mesh filename=allegro_digit/collision/digit.STL; visual mesh filename=allegro_digit/stl/digit.STL
- link link_2.0: geometry collision mesh filename=allegro_digit/collision/link_2.0_merged.STL; visual mesh filename=allegro_digit/stl/link_2.0.STL
- link link_3.0: geometry collision mesh filename=allegro_digit/collision/link_3.0_merged.STL; visual mesh filename=allegro_digit/stl/link_3.0.STL
- link link_3.0_tip: geometry collision mesh filename=allegro_digit/collision/digit.STL; visual mesh filename=allegro_digit/stl/digit.STL
- link link_4.0: geometry collision mesh filename=allegro_digit/collision/link_0.0_merged.STL; visual mesh filename=allegro_digit/stl/link_0.0.STL
- link link_5.0: geometry collision mesh filename=allegro_digit/collision/link_1.0_merged.STL; visual mesh filename=allegro_digit/stl/link_1.0.STL
- link link_6.0: geometry collision mesh filename=allegro_digit/collision/link_2.0_merged.STL; visual mesh filename=allegro_digit/stl/link_2.0.STL
- link link_7.0: geometry collision mesh filename=allegro_digit/collision/link_3.0_merged.STL; visual mesh filename=allegro_digit/stl/link_3.0.STL
- link link_7.0_tip: geometry collision mesh filename=allegro_digit/collision/digit.STL; visual mesh filename=allegro_digit/stl/digit.STL
- link link_8.0: geometry collision mesh filename=allegro_digit/collision/link_0.0_merged.STL; visual mesh filename=allegro_digit/stl/link_0.0.STL
- link link_9.0: geometry collision mesh filename=allegro_digit/collision/link_1.0_merged.STL; visual mesh filename=allegro_digit/stl/link_1.0.STL
